Commit message: Update file pathes

File: naviton/nvt_simulation/robots/naviton.urdf.xacro (robot description, xacro)
@@ -1,13 +1,13 @@
 <?xml version="1.0"?>
 <robot name="naviton" xmlns:xacro="http://ros.org/wiki/xacro">
-  <xacro:include filename="$(find kcctsim)/urdf/base/base.urdf.xacro"/>
-  <xacro:include filename="$(find kcctsim)/urdf/wheel/wheel.urdf.xacro"/>
-  <xacro:include filename="$(find kcctsim)/urdf/sensors/gps/gps.urdf.xacro"/>
-  <xacro:include filename="$(find kcctsim)/urdf/sensors/gim30/gim30.urdf.xacro"/>
-  <xacro:include filename="$(find kcctsim)/urdf/sensors/lrf/lrf.urdf.xacro"/>
+  <xacro:include filename="$(find nvt_simulation)/urdf/base/base.urdf.xacro"/>
+  <xacro:include filename="$(find nvt_simulation)/urdf/wheel/wheel.urdf.xacro"/>
+  <xacro:include filename="$(find nvt_simulation)/urdf/sensors/gps/gps.urdf.xacro"/>
+  <xacro:include filename="$(find nvt_simulation)/urdf/sensors/gim30/gim30.urdf.xacro"/>
+  <xacro:include filename="$(find nvt_simulation)/urdf/sensors/lrf/lrf.urdf.xacro"/>
   <xacro:arg name="use_nominal_extrinsics" default="false" />
   <xacro:include filename="$(find realsense2_description)/urdf/_d435i.urdf.xacro"/>
   <xacro:include filename="$(find velodyne_description)/urdf/HDL-32E.urdf.xacro"/>
-  <xacro:include filename="$(find kcctsim)/urdf/sensors/imu/imu.urdf.xacro" />
+  <xacro:include filename="$(find nvt_simulation)/urdf/sensors/imu/imu.urdf.xacro" />
   <!-- =============== Link & Joint =============== -->
   <!-- Base -->
@@ -38,6 +38,5 @@
   <!-- Front LRF -->
   <xacro:lrf_v0 prefix="front" parent="base_link">
-  	<!--origin xyz="0.225 0.0 0.195" /-->
-    <origin xyz="0.225 0.0 0.192" rpy="3.141592 0.0 0.0" />
+  	<origin xyz="0.225 0.0 0.195" />
   </xacro:lrf_v0>
   <link name="2d_blue"/>

File: naviton/nvt_simulation/urdf/base/base.urdf.xacro (robot description, xacro)
@@ -1,5 +1,5 @@
 <?xml version="1.0"?>
 <robot xmlns:xacro="http://ros.org/wiki/xacro">
-  <xacro:include filename="$(find kcctsim)/urdf/base/base.gazebo.xacro"/>
+  <xacro:include filename="$(find nvt_simulation)/urdf/base/base.gazebo.xacro"/>
   <xacro:macro name="base_v0" params="parent *joint_origin">
 	<joint name="base_link_joint" type="fixed">
@@ -11,6 +11,6 @@
 	  <visual>
 		<geometry>
-		 <!--- <mesh filename="package://kcctsim/meshes/DAE/base/base_link.dae"/>-->
-		 <mesh filename="package://kcctsim/meshes/STL/base/body.stl"/>
+		 <!--- <mesh filename="package://nvt_simulation/meshes/DAE/base/base_link.dae"/>-->
+		 <mesh filename="package://nvt_simulation/meshes/STL/base/body.stl"/>
 		</geometry>
 		<material name="gray">
@@ -20,5 +20,5 @@
 	  <collision>
 		<geometry>
-		  <mesh filename="package://kcctsim/meshes/STL/base/body.stl"/>
+		  <mesh filename="package://nvt_simulation/meshes/STL/base/body.stl"/>
 		</geometry>
 	  </collision>

File: naviton/nvt_simulation/urdf/sensors/gim30/gim30.urdf.xacro (robot description, xacro)
@@ -1,5 +1,5 @@
 <?xml version="1.0"?>
 <robot xmlns:xacro="http://ros.org/wiki/xacro">
-  <xacro:include filename="$(find kcctsim)/urdf/common.xacro"/>
+  <xacro:include filename="$(find nvt_simulation)/urdf/common.xacro"/>
   <xacro:macro name="gim30_v0" params="parent *joint_origin">
 	<joint name="gim30_joint" type="fixed">
@@ -11,10 +11,10 @@
       <visual>
         <geometry>
-          <mesh filename="package://kcctsim/meshes/DAE/sensors/gim30/gim30.dae"/>
+          <mesh filename="package://nvt_simulation/meshes/DAE/sensors/gim30/gim30.dae"/>
         </geometry>
       </visual>
 	  <collision>
 		<geometry>
-		  <mesh filename="package://kcctsim/meshes/STL/sensors/gim30/gim30.stl"/>
+		  <mesh filename="package://nvt_simulation/meshes/STL/sensors/gim30/gim30.stl"/>
 		</geometry>
 	  </collision>

File: naviton/nvt_simulation/urdf/sensors/gps/gps.urdf.xacro (robot description, xacro)
@@ -1,5 +1,5 @@
 <?xml version="1.0"?>
 <robot xmlns:xacro="http://ros.org/wiki/xacro">
-  <xacro:include filename="$(find kcctsim)/urdf/common.xacro"/>
+  <xacro:include filename="$(find nvt_simulation)/urdf/common.xacro"/>
   <xacro:macro name="gps_v0" params="parent *joint_origin">
 	<joint name="gps_joint" type="fixed">
@@ -11,10 +11,10 @@
 	  <visual>
 		<geometry>
-		  <mesh filename="package://kcctsim/meshes/DAE/sensors/gps/gps.dae"/>
+		  <mesh filename="package://nvt_simulation/meshes/DAE/sensors/gps/gps.dae"/>
 		</geometry>
 	  </visual>
 	  <collision>
 		<geometry>
-		  <mesh filename="package://kcctsim/meshes/STL/sensors/gps/gps.stl"/>
+		  <mesh filename="package://nvt_simulation/meshes/STL/sensors/gps/gps.stl"/>
 		</geometry>
 	  </collision>

File: naviton/nvt_simulation/urdf/sensors/lrf/lrf.urdf.xacro (robot description, xacro)
@@ -1,6 +1,6 @@
 <?xml version="1.0"?>
 <robot xmlns:xacro="http://ros.org/wiki/xacro">
-  <xacro:include filename="$(find kcctsim)/urdf/common.xacro"/>
-  <xacro:include filename="$(find kcctsim)/urdf/sensors/lrf/lrf.gazebo.xacro"/>
+  <xacro:include filename="$(find nvt_simulation)/urdf/common.xacro"/>
+  <xacro:include filename="$(find nvt_simulation)/urdf/sensors/lrf/lrf.gazebo.xacro"/>
   <xacro:macro name="lrf_v0" params="prefix parent *joint_origin">
 	<joint name="${prefix}_lrf_joint" type="fixed">
@@ -12,10 +12,10 @@
 	  <visual>
 		<geometry>
-		  <mesh filename="package://kcctsim/meshes/STL/sensors/utm30lx.stl"/>
+		  <mesh filename="package://nvt_simulation/meshes/STL/sensors/utm30lx.stl"/>
 		</geometry>
 	  </visual>
 	  <collision>
 		<geometry>
-		  <mesh filename="package://kcctsim/meshes/STL/sensors/utm30lx.stl"/>
+		  <mesh filename="package://nvt_simulation/meshes/STL/sensors/utm30lx.stl"/>
 		</geometry>
 	  </collision>

File: naviton/nvt_simulation/urdf/wheel/wheel.urdf.xacro (robot description, xacro)
@@ -1,7 +1,7 @@
 <?xml version="1.0"?>
 <robot xmlns:xacro="http://ros.org/wiki/xacro">
-  <xacro:include filename="$(find kcctsim)/urdf/common.xacro"/>
-  <xacro:include filename="$(find kcctsim)/urdf/wheel/wheel.transmission.xacro"/>
-  <xacro:include filename="$(find kcctsim)/urdf/wheel/wheel.gazebo.xacro"/>
+  <xacro:include filename="$(find nvt_simulation)/urdf/common.xacro"/>
+  <xacro:include filename="$(find nvt_simulation)/urdf/wheel/wheel.transmission.xacro"/>
+  <xacro:include filename="$(find nvt_simulation)/urdf/wheel/wheel.gazebo.xacro"/>
   <property name="wheel_radius" value="0.1575"/>
   <property name="wheel_length" value="0.032"/>
@@ -17,6 +17,6 @@
 	  <visual>
 		<geometry>
-		  <!--<mesh filename="package://kcctsim/meshes/DAE/wheel/wheel_link.dae"/>-->
-		   <mesh filename="package://kcctsim/meshes/STL/wheel/wheel.stl"/>
+		  <!--<mesh filename="package://nvt_simulation/meshes/DAE/wheel/wheel_link.dae"/>-->
+		   <mesh filename="package://nvt_simulation/meshes/STL/wheel/wheel.stl"/>
 		</geometry>
 		<material name="black">

Commit message: Create sensorless robot model

File: naviton/nvt_simulation/robots/naviton.urdf.xacro (robot description, xacro)
@@ -1,103 +1,39 @@
 <?xml version="1.0"?>
 <robot name="naviton" xmlns:xacro="http://ros.org/wiki/xacro">
-  <xacro:include filename="$(find nvt_simulation)/urdf/base/base.urdf.xacro"/>
-  <xacro:include filename="$(find nvt_simulation)/urdf/wheel/wheel.urdf.xacro"/>
-  <xacro:include filename="$(find nvt_simulation)/urdf/sensors/gps/gps.urdf.xacro"/>
-  <xacro:include filename="$(find nvt_simulation)/urdf/sensors/gim30/gim30.urdf.xacro"/>
-  <xacro:include filename="$(find nvt_simulation)/urdf/sensors/lrf/lrf.urdf.xacro"/>
-  <xacro:arg name="use_nominal_extrinsics" default="false" />
-  <xacro:include filename="$(find realsense2_description)/urdf/_d435i.urdf.xacro"/>
-  <xacro:include filename="$(find velodyne_description)/urdf/HDL-32E.urdf.xacro"/>
-  <xacro:include filename="$(find nvt_simulation)/urdf/sensors/imu/imu.urdf.xacro" />
-  <!-- =============== Link & Joint =============== -->
-  <!-- Base -->
-  <link name="base_link"/>
-  <xacro:base_v0 parent="base_link">
-	<origin xyz="0 0 0.0"/>
-  </xacro:base_v0>
-  <!-- Wheel -->
-  <!-- Right Wheel -->
-  <xacro:wheel_v0 prefix="right" parent="base_link">
-	<origin xyz="0 -0.2775 0.1575"/>
-	<axis xyz="0 1 0"/>
-  </xacro:wheel_v0>
-  <!-- Left Wheel -->
-  <xacro:wheel_v0 prefix="left" parent="base_link">
-	<origin xyz="0 0.2775 0.1575" rpy="0 0 ${M_PI}"/>
-	<axis xyz="0 -1 0"/>
-  </xacro:wheel_v0>
-  <!-- Sensors -->
-  <!-- GPS -->
- <!--- <xacro:gps_v0 parent="base_link">
-	<origin xyz="-0.06229 0 0.420552" rpy="0 0 -${M_PI}"/>
-  </xacro:gps_v0>-->
-  <!-- Gim30 -->
- <!--<xacro:gim30_v0 parent="base_link">
-  	<origin xyz="0.07395931 0 0.24578237"/>
-  </xacro:gim30_v0>-->
-  <!-- Front LRF -->
-  <xacro:lrf_v0 prefix="front" parent="base_link">
-  	<origin xyz="0.225 0.0 0.195" />
-  </xacro:lrf_v0>
-  <link name="2d_blue"/>
-    <joint name="2d_blue_joint" type="fixed">
-    <parent link="front_lrf_link"/>
-    <child link="2d_blue"/>
-    <origin xyz="0 0 0"/>
-  </joint>
-  <!-- Rear LRF -->
-  <xacro:lrf_v0 prefix="rear" parent="base_link">
-  	<origin xyz="-0.485 0.0 0.195" rpy="0 0 -${M_PI}"/>
-  </xacro:lrf_v0>
-  <link name="2d_orange"/>
-    <joint name="2d_orange_joint" type="fixed">
-    <parent link="rear_lrf_link"/>
-    <child link="2d_orange"/>
-    <origin xyz="0 0 0"/>
-  </joint>
-  <link name="camera_link"/>
-    <joint name="lrf_link_joint" type="fixed">
-    <parent link="base_link"/>
-    <child link="camera_link"/>
-    <origin xyz="0 0 0.195"/>
-  </joint>
-<!--
-  <link name="imu_link"/>
-  <joint name="imu_link_joint" type="fixed">
-	<parent link="base_link"/>
-	<child link="imu_link"/>
-	<origin xyz="0 0 0.051" rpy="0 0 0" />
-  </joint>-->
-  <!-- ===============  Transmission =============== -->
-  <xacro:wheel_trans_v0 prefix="right"/>
-  <xacro:wheel_trans_v0 prefix="left"/>
-  <!-- =============== Gazebo =============== -->
-  <gazebo>
-    <plugin name="gazebo_ros_control" filename="libgazebo_ros_control.so">
-      <!-- <robotNamespace>fourth_robot</robotNamespace> -->
-    </plugin>
-  </gazebo>
-  <!-- Base -->
-  <xacro:base_gazebo_v0/>
-  <!-- Wheel -->
-  <xacro:wheel_gazebo_v0 prefix="right"/>
-  <xacro:wheel_gazebo_v0 prefix="left"/>
-  <!-- <xacro:wheel_gazebo_control_v0 rate="25"/> -->
-  <!--IMU-->
-  <xacro:imu_macro prefix="imu" parent="base_link" xyz="0 0 0"/>
-  <!-- LRF -->
-  <xacro:lrf_gazebo_v0 topic_name="scan1" prefix="front"
-					   min_rad="-1.65806278939" max_rad="1.65806278939"
-					   min_range="0.10" max_range="60.0" />
-  <xacro:lrf_gazebo_v0 topic_name="scan2" prefix="rear"
-					   min_rad="-1.65806278939" max_rad="1.65619449019"
-					   min_range="0.10" max_range="60.0"/>
-  <!-- Realsense -->
-  <xacro:sensor_d435i parent="base_link" name="d435i" use_nominal_extrinsics="$(arg use_nominal_extrinsics)">
-    <origin xyz="0.035 0 0.665" rpy="0 0.7854 0" />
-  </xacro:sensor_d435i>
-  <!-- VHDL-32E -->
-  <HDL-32E parent="base_link" name="velodyne_link" topic="velodyne_points" hz="10" samples="1024" gpu="true">
-      <origin xyz="-0.1 0 0.8" rpy="0 0 0" />
-  </HDL-32E>
+    <!-- ======== Include ======== -->
+    <xacro:include filename="$(find nvt_simulation)/urdf/base/base.urdf.xacro" />
+    <xacro:include filename="$(find nvt_simulation)/urdf/wheel/wheel.urdf.xacro" />
+    <xacro:include filename="$(find nvt_simulation)/urdf/wheel/wheel.transmission.xacro" />
+    <!--xacro:include filename="$(find nvt_simulation)/urdf/sensors/lrf/lrf.urdf.xacro" />
+    <xacro:include filename="$(find velodyne_description)/urdf/HDL-32E.urdf.xacro" />
+    <xacro:include filename="$(find nvt_simulation)/urdf/sensors/imu/imu.urdf.xacro" /-->
+    <!-- ======== Gazebo ======== -->
+    <gazebo>
+        <plugin name="gazebo_ros_control" filename="libgazebo_ros_control.so" />
+        <robotNamespace> /naviton </robotNamespace>
+        <robotSimType> gazebo_ros_control/DefaultRobotHWSim </robotSimType>
+        <robotParam> /naviton/robot_description </robotParam>
+        <legacyModeNS> true </legacyModeNS>
+    </gazebo>
+    <!-- ======== Base ======== -->
+    <link name="base_link"/>
+    <xacro:base_v0 parent="base_link">
+	    <origin xyz="0 0 0"/>
+    </xacro:base_v0>
+    <xacro:base_gazebo_v0 />
+    <!-- ======== Wheel ======== -->
+    <!-- Right -->
+    <xacro:wheel_v0 prefix="right" parent="base_link">
+	    <origin xyz="0 -0.2775 0.1575"/>
+	    <axis xyz="0 1 0"/>
+    </xacro:wheel_v0>
+    <xacro:wheel_trans_v0 prefix="right" />
+    <xacro:wheel_gazebo_v0 prefix="right" />
+    <!-- Left -->
+    <xacro:wheel_v0 prefix="left" parent="base_link">
+	    <origin xyz="0 0.2775 0.1575" rpy="0 0 ${M_PI}"/>
+	    <axis xyz="0 -1 0"/>
+    </xacro:wheel_v0>
+    <xacro:wheel_trans_v0 prefix="left" />
+    <xacro:wheel_gazebo_v0 prefix="left" />
 </robot>

File: naviton/nvt_simulation/urdf/base/base.gazebo.xacro (robot description, xacro)
@@ -2,6 +2,6 @@
 <robot xmlns:xacro="http://ros.org/wiki/xacro">
   <xacro:macro name="base_gazebo_v0">
-	<gazebo reference="base_link">
-	  <selfCollide>false</selfCollide>
+	  <gazebo reference="base_link">
+	    <selfCollide> false </selfCollide>
       <mu1 value="0.05" />
       <mu2 value="0.05" />

File: naviton/nvt_simulation/urdf/base/base.urdf.xacro (robot description, xacro)
@@ -1,34 +1,31 @@
 <?xml version="1.0"?>
 <robot xmlns:xacro="http://ros.org/wiki/xacro">
-  <xacro:include filename="$(find nvt_simulation)/urdf/base/base.gazebo.xacro"/>
-  <xacro:macro name="base_v0" params="parent *joint_origin">
-	<joint name="base_link_joint" type="fixed">
-	  <insert_block name="joint_origin"/>
-	  <parent link="${parent}"/>
-	  <child link="body_link"/>
-	</joint>
-	<link name="body_link">
-	  <visual>
-		<geometry>
-		 <!--- <mesh filename="package://nvt_simulation/meshes/DAE/base/base_link.dae"/>-->
-		 <mesh filename="package://nvt_simulation/meshes/STL/base/body.stl"/>
-		</geometry>
-		<material name="gray">
-    <color rgba="0.8 0.8 0.8 2.0"/>
-  </material>
-	  </visual>
-	  <collision>
-		<geometry>
-		  <mesh filename="package://nvt_simulation/meshes/STL/base/body.stl"/>
-		</geometry>
-	  </collision>
-	  <inertial>
-		<origin xyz="-0.061 0 -0.002"/>
-		<mass value="45"/>
-		<inertia ixx="1.64890" ixy="0" ixz="-0.21424"
-				 iyy="2.24766" iyz="0"
-				 izz="1.25664" />
-	  </inertial>
-	</link>
-  </xacro:macro>
+	<xacro:include filename="$(find nvt_simulation)/urdf/base/base.gazebo.xacro"/>
+	<xacro:macro name="base_v0" params="parent *joint_origin">
+		<joint name="base_link_joint" type="fixed">
+			<insert_block name="joint_origin"/>
+			<parent link="${parent}"/>
+			<child link="body_link"/>
+		</joint>
+		<link name="body_link">
+			<visual>
+				<geometry>
+					<mesh filename="package://nvt_simulation/meshes/STL/base/body.stl"/>
+				</geometry>
+				<material name="gray">
+    				<color rgba="0.8 0.8 0.8 2.0"/>
+  				</material>
+	  		</visual>
+			<collision>
+				<geometry>
+		  			<mesh filename="package://nvt_simulation/meshes/STL/base/body.stl"/>
+				</geometry>
+			</collision>
+			<inertial>
+				<origin xyz="-0.061 0 -0.002"/>
+				<mass value="45"/>
+				<inertia ixx="1.64890" ixy="0" ixz="-0.21424" iyy="2.24766" iyz="0" izz="1.25664" />
+	  		</inertial>
+		</link>
+	</xacro:macro>
 </robot>

File: naviton/nvt_simulation/urdf/wheel/wheel.gazebo.xacro (robot description, xacro)
@@ -2,6 +2,6 @@
 <robot xmlns:xacro="http://ros.org/wiki/xacro">
   <xacro:macro name="wheel_gazebo_v0" params="prefix">
-	<gazebo reference="${prefix}_wheel_link">
-	  <selfCollide>false</selfCollide>
+	  <gazebo reference="${prefix}_wheel_link">
+	    <selfCollide> false </selfCollide>
       <mu1 value="0.8" />
       <mu2 value="0.8" />

File: naviton/nvt_simulation/urdf/wheel/wheel.transmission.xacro (robot description, xacro)
@@ -2,14 +2,14 @@
 <robot xmlns:xacro="http://ros.org/wiki/xacro">
   <xacro:macro name="wheel_trans_v0" params="prefix">
-	<transmission name="${prefix}_wheel_trans">
-      <type>transmission_interface/SimpleTransmission</type>
+    <transmission name="${prefix}_wheel_trans">
+      <type> transmission_interface/SimpleTransmission </type>
       <joint name="${prefix}_wheel_joint">
-		<hardwareInterface>VelocityJointInterface</hardwareInterface>
+	      <hardwareInterface>VelocityJointInterface</hardwareInterface>
       </joint>
-	  <actuator name="${prefix}_wheel_motor">
-		<hardwareInterface>VelocityJointInterface</hardwareInterface>
-		<mechanicalReduction>30</mechanicalReduction>
+      <actuator name="${prefix}_wheel_motor">
+        <hardwareInterface> VelocityJointInterface </hardwareInterface>
+        <mechanicalReduction> 30 </mechanicalReduction>
       </actuator>
-	</transmission>
+    </transmission>
   </xacro:macro>
 </robot>

File: naviton/nvt_simulation/urdf/wheel/wheel.urdf.xacro (robot description, xacro)
@@ -1,39 +1,37 @@
 <?xml version="1.0"?>
 <robot xmlns:xacro="http://ros.org/wiki/xacro">
-  <xacro:include filename="$(find nvt_simulation)/urdf/common.xacro"/>
-  <xacro:include filename="$(find nvt_simulation)/urdf/wheel/wheel.transmission.xacro"/>
-  <xacro:include filename="$(find nvt_simulation)/urdf/wheel/wheel.gazebo.xacro"/>
-  <property name="wheel_radius" value="0.1575"/>
-  <property name="wheel_length" value="0.032"/>
-  <property name="wheel_mass" value="2.0"/>
-  <xacro:macro name="wheel_v0" params="prefix parent *joint_origin *joint_axis">
-	<joint name="${prefix}_wheel_joint" type="continuous">
-	  <insert_block name="joint_origin"/>
-	  <parent link="${parent}"/>
-	  <child link="${prefix}_wheel_link"/>
-	  <insert_block name="joint_axis"/>
-	</joint>
-	<link name="${prefix}_wheel_link">
-	  <visual>
-		<geometry>
-		  <!--<mesh filename="package://nvt_simulation/meshes/DAE/wheel/wheel_link.dae"/>-->
-		   <mesh filename="package://nvt_simulation/meshes/STL/wheel/wheel.stl"/>
-		</geometry>
-		<material name="black">
-    		<color rgba="0.2 0.2 0.2 2.0"/>
-  		</material>
-	  </visual>
-	  <collision>
-		<origin xyz="0 -0.003 0" rpy="${-M_PI/2} 0 0"/>
-		<geometry>
-		  <cylinder radius="${wheel_radius}" length="${wheel_length}"/>
-		</geometry>
-	  </collision>
-	  <inertial>
-		<origin xyz="0 -0.003 0" rpy="${-M_PI/2} 0 0"/>
-		<cylinder_inertial mass="${wheel_mass}"
+    <xacro:include filename="$(find nvt_simulation)/urdf/utils.xacro" />
+    <xacro:include filename="$(find nvt_simulation)/urdf/wheel/wheel.gazebo.xacro"/>
+    <property name="wheel_radius" value="0.1575"/>
+    <property name="wheel_length" value="0.032"/>
+    <property name="wheel_mass" value="2.0"/>
+    <xacro:macro name="wheel_v0" params="prefix parent *joint_origin *joint_axis">
+        <joint name="${prefix}_wheel_joint" type="continuous">
+	        <insert_block name="joint_origin"/>
+	        <parent link="${parent}"/>
+	        <child link="${prefix}_wheel_link"/>
+	        <insert_block name="joint_axis"/>
+	    </joint>
+        <link name="${prefix}_wheel_link">
+            <visual>
+		        <geometry>
+		            <mesh filename="package://nvt_simulation/meshes/STL/wheel/wheel.stl"/>
+		        </geometry>
+                <material name="black">
+    		        <color rgba="0.2 0.2 0.2 2.0"/>
+                </material>
+	        </visual>
+            <collision>
+		        <origin xyz="0 -0.003 0" rpy="${-M_PI/2} 0 0"/>
+		        <geometry>
+		            <cylinder radius="${wheel_radius}" length="${wheel_length}"/>
+		        </geometry>
+	        </collision>
+            <inertial>
+		        <origin xyz="0 -0.003 0" rpy="${-M_PI/2} 0 0"/>
+		        <cylinder_inertial mass="${wheel_mass}"
 						   radius="${wheel_radius}" length="${wheel_length}"/>
-	  </inertial>
-	</link>
-  </xacro:macro>
+	        </inertial>
+        </link>
+    </xacro:macro>
 </robot>
