Commit message: nvt_description package

File: naviton/nvt_description/base.urdf.xacro (robot description, xacro)
@@ -1,5 +1,5 @@
 <?xml version="1.0"?>
 <robot xmlns:xacro="http://ros.org/wiki/xacro">
-	<xacro:include filename="$(find nvt_simulation)/urdf/base/base.gazebo.xacro"/>
+	<!--xacro:include filename="$(find nvt_description)/urdf/base/base.gazebo.xacro"/>
 	<xacro:macro name="base_v0" params="parent *joint_origin">
 		<joint name="base_link_joint" type="fixed">
@@ -11,5 +11,5 @@
 			<visual>
 				<geometry>
-					<mesh filename="package://nvt_simulation/meshes/STL/base/body.stl"/>
+					<mesh filename="package://nvt_description/meshes/STL/base/body.stl"/>
 				</geometry>
 				<material name="gray">
@@ -19,5 +19,5 @@
 			<collision>
 				<geometry>
-		  			<mesh filename="package://nvt_simulation/meshes/STL/base/body.stl"/>
+		  			<mesh filename="package://nvt_description/meshes/STL/base/body.stl"/>
 				</geometry>
 			</collision>
@@ -28,4 +28,4 @@
 	  		</inertial>
 		</link>
-	</xacro:macro>
+	</xacro:macro-->
 </robot>

File: naviton/nvt_description/urdf/naviton.urdf.xacro (robot description, xacro)
@@ -1,8 +1,10 @@
 <?xml version="1.0"?>
-<robot name="naviton" xmlns:xacro="http://ros.org/wiki/xacro">
+<robot xmlns:xacro="http://ros.org/wiki/xacro" name="naviton">
+    <xacro:property name="package_name" value="nvt_description" />
+    <xacro:property name="robot_name" value="naviton" />
     <!-- ======== Include ======== -->
-    <xacro:include filename="$(find nvt_simulation)/urdf/base/base.urdf.xacro" />
-    <xacro:include filename="$(find nvt_simulation)/urdf/wheel/wheel.urdf.xacro" />
-    <xacro:include filename="$(find nvt_simulation)/urdf/wheel/wheel.transmission.xacro" />
+    <xacro:include filename="$(find ${package_name})/urdf/base/base.urdf.xacro" />
+    <xacro:include filename="$(find ${package_name})/urdf/wheel/wheel.urdf.xacro" />
+    <xacro:include filename="$(find ${package_name})/urdf/wheel/wheel.transmission.xacro" />
     <!--xacro:include filename="$(find nvt_simulation)/urdf/sensors/lrf/lrf.urdf.xacro" />
     <xacro:include filename="$(find velodyne_description)/urdf/HDL-32E.urdf.xacro" />

File: naviton/nvt_description/urdf/utils/inertia.xacro (robot description, xacro)
@@ -1,6 +1,8 @@
 <?xml version="1.0"?>
 <robot xmlns:xacro="http://ros.org/wiki/xacro">
+	<!-- ====== Constant Values ====== -->
 	<property name="M_PI" value="3.14159265"/>
-	<xacro:macro name="cylinder_inertial" params="mass radius length">
+	<!-- ====== Inertia ====== -->
+	<xacro:macro name="cylinder_inertia" params="mass radius length">
 		<mass value="${mass}"/>
 		<inertia 	ixx="${((radius*radius)/4 + (length*length)/12)*mass}" ixy="0" ixz="0"
@@ -8,5 +10,5 @@
 					izz="${(mass*radius*radius)/2}" />
   	</xacro:macro>
-	<xacro:macro name="box_inertial" params="mass height width depth">
+	<xacro:macro name="box_inertia" params="mass height width depth">
 		<mass value="${mass}"/>
 		<inertia 	ixx="${(mass*(width*width+depth*depth))/12}"	ixy="0" ixz="0"

File: naviton/nvt_description/urdf/wheel/wheel.urdf.xacro (robot description, xacro)
@@ -1,6 +1,6 @@
 <?xml version="1.0"?>
 <robot xmlns:xacro="http://ros.org/wiki/xacro">
-    <xacro:include filename="$(find nvt_simulation)/urdf/utils.xacro" />
-    <xacro:include filename="$(find nvt_simulation)/urdf/wheel/wheel.gazebo.xacro"/>
+    <xacro:include filename="$(find nvt_description)/urdf/utils/inertia.xacro" />
+    <xacro:include filename="$(find nvt_description)/urdf/wheel/wheel.gazebo.xacro"/>
     <property name="wheel_radius" value="0.1575"/>
     <property name="wheel_length" value="0.032"/>
@@ -16,5 +16,5 @@
             <visual>
 		        <geometry>
-		            <mesh filename="package://nvt_simulation/meshes/STL/wheel/wheel.stl"/>
+		            <mesh filename="package://nvt_description/meshes/STL/wheel/wheel.stl"/>
 		        </geometry>
                 <material name="black">
@@ -30,5 +30,5 @@
             <inertial>
 		        <origin xyz="0 -0.003 0" rpy="${-M_PI/2} 0 0"/>
-		        <cylinder_inertial mass="${wheel_mass}"
+		        <cylinder_inertia mass="${wheel_mass}"
 						   radius="${wheel_radius}" length="${wheel_length}"/>
 	        </inertial>
