Commit message: Fix xacro tags

File: naviton/nvt_description/urdf/base/base.urdf.xacro (robot description, xacro)
@@ -4,5 +4,5 @@
 	<xacro:macro name="base_v0" params="parent *joint_origin">
 		<joint name="base_link_joint" type="fixed">
-			<insert_block name="joint_origin"/>
+			<xacro:insert_block name="joint_origin"/>
 			<parent link="${parent}"/>
 			<child link="body_link"/>

File: naviton/nvt_description/urdf/naviton.urdf.xacro (robot description, xacro)
@@ -33,7 +33,7 @@
     <!-- ======== Sensors ======== -->
     <!-- VHDL-32E -->
-    <HDL-32E parent="base_link" name="velodyne_link" topic="velodyne_points/raw" hz="10" samples="1024" gpu="true">
+    <xacro:HDL-32E parent="base_link" name="velodyne_link" topic="velodyne_points/raw" hz="10" samples="1024" gpu="true">
         <origin xyz="0 0 0.8" rpy="0 0 0" />
-    </HDL-32E>
+    </xacro:HDL-32E>
     <!-- LRF -->
     <xacro:lrf_v0 prefix="front" parent="base_link">

File: naviton/nvt_description/urdf/sensors/gim30/gim30.urdf.xacro (robot description, xacro)
@@ -4,5 +4,5 @@
   <xacro:macro name="gim30_v0" params="parent *joint_origin">
 	<joint name="gim30_joint" type="fixed">
-      <insert_block name="joint_origin" />
+      <xacro:insert_block name="joint_origin" />
       <parent link="${parent}"/>
       <child link="gim30_link"/>

File: naviton/nvt_description/urdf/sensors/gps/gps.urdf.xacro (robot description, xacro)
@@ -4,5 +4,5 @@
   <xacro:macro name="gps_v0" params="parent *joint_origin">
 	<joint name="gps_joint" type="fixed">
-	  <insert_block name="joint_origin"/>
+	  <xacro:insert_block name="joint_origin"/>
 	  <parent link="${parent}"/>
 	  <child link="gps_link"/>

File: naviton/nvt_description/urdf/sensors/lrf/lrf.urdf.xacro (robot description, xacro)
@@ -5,5 +5,5 @@
   <xacro:macro name="lrf_v0" params="prefix parent *joint_origin">
 	<joint name="${prefix}_lrf_joint" type="fixed">
-	  <insert_block name="joint_origin"/>
+	  <xacro:insert_block name="joint_origin"/>
 	  <parent link="${parent}"/>
 	  <child link="${prefix}_lrf_link"/>
@@ -22,5 +22,5 @@
 	  <inertial>
 		<origin xyz="0 0 -0.0164"/>
-		<box_inertia mass="0.4" height="0.07" width="0.07" depth="0.08"/>
+		<xacro:box_inertia mass="0.4" height="0.07" width="0.07" depth="0.08"/>
 	  </inertial>
 	</link>

File: naviton/nvt_description/urdf/utils/inertia.xacro (robot description, xacro)
@@ -2,5 +2,5 @@
 <robot xmlns:xacro="http://ros.org/wiki/xacro">
 	<!-- ====== Constant Values ====== -->
-	<property name="M_PI" value="3.14159265"/>
+	<xacro:property name="M_PI" value="3.14159265"/>
 	<!-- ====== Inertia ====== -->
 	<xacro:macro name="cylinder_inertia" params="mass radius length">

File: naviton/nvt_description/urdf/wheel/wheel.urdf.xacro (robot description, xacro)
@@ -3,13 +3,13 @@
     <xacro:include filename="$(find nvt_description)/urdf/utils/inertia.xacro" />
     <xacro:include filename="$(find nvt_description)/urdf/wheel/wheel.gazebo.xacro"/>
-    <property name="wheel_radius" value="0.1575"/>
-    <property name="wheel_length" value="0.032"/>
-    <property name="wheel_mass" value="2.0"/>
+    <xacro:property name="wheel_radius" value="0.1575"/>
+    <xacro:property name="wheel_length" value="0.032"/>
+    <xacro:property name="wheel_mass" value="2.0"/>
     <xacro:macro name="wheel_v0" params="prefix parent *joint_origin *joint_axis">
         <joint name="${prefix}_wheel_joint" type="continuous">
-	        <insert_block name="joint_origin"/>
+	        <xacro:insert_block name="joint_origin"/>
 	        <parent link="${parent}"/>
 	        <child link="${prefix}_wheel_link"/>
-	        <insert_block name="joint_axis"/>
+	        <xacro:insert_block name="joint_axis"/>
 	    </joint>
         <link name="${prefix}_wheel_link">
@@ -30,5 +30,5 @@
             <inertial>
 		        <origin xyz="0 -0.003 0" rpy="${-M_PI/2} 0 0"/>
-		        <cylinder_inertia mass="${wheel_mass}"
+		        <xacro:cylinder_inertia mass="${wheel_mass}"
 						   radius="${wheel_radius}" length="${wheel_length}"/>
 	        </inertial>

Commit message: Fix xacro colors

File: naviton/nvt_description/urdf/base/base.urdf.xacro (robot description, xacro)
@@ -14,5 +14,5 @@
 				</geometry>
 				<material name="gray">
-    				<color rgba="0.8 0.8 0.8 2.0"/>
+    				<color rgba="0.8 0.8 0.8 1.0"/>
   				</material>
 	  		</visual>

File: naviton/nvt_description/urdf/sensors/lrf/lrf.urdf.xacro (robot description, xacro)
@@ -14,4 +14,7 @@
 		  <mesh filename="package://nvt_description/meshes/STL/sensors/utm30lx.stl"/>
 		</geometry>
+		<material name="black">
+    	  <color rgba="0.2 0.2 0.2 1.0"/>
+        </material>
 	  </visual>
 	  <collision>

File: naviton/nvt_description/urdf/wheel/wheel.urdf.xacro (robot description, xacro)
@@ -19,5 +19,5 @@
 		        </geometry>
                 <material name="black">
-    		        <color rgba="0.2 0.2 0.2 2.0"/>
+    		        <color rgba="0.2 0.2 0.2 1.0"/>
                 </material>
 	        </visual>
