Commit message: Add hdl32e to urdf

File: naviton/nvt_description/urdf/naviton.urdf.xacro (robot description, xacro)
@@ -7,7 +7,7 @@
     <xacro:include filename="$(find ${package_name})/urdf/wheel/wheel.urdf.xacro" />
     <xacro:include filename="$(find ${package_name})/urdf/wheel/wheel.transmission.xacro" />
-    <!--xacro:include filename="$(find nvt_simulation)/urdf/sensors/lrf/lrf.urdf.xacro" />
+    <!--xacro:include filename="$(find nvt_simulation)/urdf/sensors/lrf/lrf.urdf.xacro" /-->
     <xacro:include filename="$(find velodyne_description)/urdf/HDL-32E.urdf.xacro" />
-    <xacro:include filename="$(find nvt_simulation)/urdf/sensors/imu/imu.urdf.xacro" /-->
+    <!-- xacro:include filename="$(find nvt_simulation)/urdf/sensors/imu/imu.urdf.xacro" /-->
     <!-- ======== Base ======== -->
     <link name="base_link"/>
@@ -16,5 +16,5 @@
     </xacro:base_v0>
     <xacro:base_gazebo_v0 />
-    <!-- ======== Wheel ======== -->
+    <!-- ======== Wheels ======== -->
     <!-- Right -->
     <xacro:wheel_v0 prefix="right" parent="base_link">
@@ -31,4 +31,9 @@
     <xacro:wheel_trans_v0 prefix="left" />
     <xacro:wheel_gazebo_v0 prefix="left" />
+    <!-- ======== Sensors ======== -->
+    <!-- VHDL-32E -->
+    <HDL-32E parent="base_link" name="velodyne_link" topic="velodyne_points" hz="10" samples="1024" gpu="true">
+        <origin xyz="0 0 0.8" rpy="0 0 0" />
+    </HDL-32E>
     <!-- ======== Gazebo ======== -->
     <gazebo>

Commit message: Add lrf scan to simulation

File: naviton/nvt_description/urdf/naviton.urdf.xacro (robot description, xacro)
@@ -7,6 +7,6 @@
     <xacro:include filename="$(find ${package_name})/urdf/wheel/wheel.urdf.xacro" />
     <xacro:include filename="$(find ${package_name})/urdf/wheel/wheel.transmission.xacro" />
-    <!--xacro:include filename="$(find nvt_simulation)/urdf/sensors/lrf/lrf.urdf.xacro" /-->
     <xacro:include filename="$(find velodyne_description)/urdf/HDL-32E.urdf.xacro" />
+    <xacro:include filename="$(find ${package_name})/urdf/sensors/lrf/lrf.urdf.xacro" />
     <!-- xacro:include filename="$(find nvt_simulation)/urdf/sensors/imu/imu.urdf.xacro" /-->
     <!-- ======== Base ======== -->
@@ -36,4 +36,11 @@
         <origin xyz="0 0 0.8" rpy="0 0 0" />
     </HDL-32E>
+    <!-- LRF -->
+    <xacro:lrf_v0 prefix="front" parent="base_link">
+  	    <origin xyz="0.225 0.0 0.195" />
+    </xacro:lrf_v0>
+    <xacro:lrf_gazebo_v0    topic_name="/lrf_scan/front" prefix="front"
+					        min_rad="-1.65806278939" max_rad="1.65806278939"
+					        min_range="0.10" max_range="60.0" />
     <!-- ======== Gazebo ======== -->
     <gazebo>

File: naviton/nvt_description/urdf/sensors/lrf/lrf.urdf.xacro (robot description, xacro)
@@ -1,6 +1,6 @@
 <?xml version="1.0"?>
 <robot xmlns:xacro="http://ros.org/wiki/xacro">
-  <xacro:include filename="$(find nvt_simulation)/urdf/common.xacro"/>
-  <xacro:include filename="$(find nvt_simulation)/urdf/sensors/lrf/lrf.gazebo.xacro"/>
+  <xacro:include filename="$(find nvt_description)/urdf/utils/inertia.xacro"/>
+  <xacro:include filename="$(find nvt_description)/urdf/sensors/lrf/lrf.gazebo.xacro"/>
   <xacro:macro name="lrf_v0" params="prefix parent *joint_origin">
 	<joint name="${prefix}_lrf_joint" type="fixed">
@@ -12,15 +12,15 @@
 	  <visual>
 		<geometry>
-		  <mesh filename="package://nvt_simulation/meshes/STL/sensors/utm30lx.stl"/>
+		  <mesh filename="package://nvt_description/meshes/STL/sensors/utm30lx.stl"/>
 		</geometry>
 	  </visual>
 	  <collision>
 		<geometry>
-		  <mesh filename="package://nvt_simulation/meshes/STL/sensors/utm30lx.stl"/>
+		  <mesh filename="package://nvt_description/meshes/STL/sensors/utm30lx.stl"/>
 		</geometry>
 	  </collision>
 	  <inertial>
 		<origin xyz="0 0 -0.0164"/>
-		<box_inertial mass="0.4" height="0.07" width="0.07" depth="0.08"/>
+		<box_inertia mass="0.4" height="0.07" width="0.07" depth="0.08"/>
 	  </inertial>
 	</link>

Commit message: Update robot model

File: naviton/nvt_description/urdf/naviton.urdf.xacro (robot description, xacro)
@@ -19,5 +19,5 @@
     <!-- Right -->
     <xacro:wheel_v0 prefix="right" parent="base_link">
-	    <origin xyz="0 -0.2775 0.1575"/>
+	    <origin xyz="0 -0.265 0.1575"/>
 	    <axis xyz="0 1 0"/>
     </xacro:wheel_v0>
@@ -26,5 +26,5 @@
     <!-- Left -->
     <xacro:wheel_v0 prefix="left" parent="base_link">
-	    <origin xyz="0 0.2775 0.1575" rpy="0 0 ${M_PI}"/>
+	    <origin xyz="0 0.265 0.1575" rpy="0 0 ${M_PI}"/>
 	    <axis xyz="0 -1 0"/>
     </xacro:wheel_v0>
@@ -38,5 +38,5 @@
     <!-- LRF -->
     <xacro:lrf_v0 prefix="front" parent="base_link">
-  	    <origin xyz="0.225 0.0 0.195" />
+  	    <origin xyz="0.155 0.0 0.195" rpy="${M_PI} 0 0"/>
     </xacro:lrf_v0>
     <xacro:lrf_gazebo_v0    topic_name="sensors/lrf/scan" prefix="front"

Commit message: Update urdf

File: naviton/nvt_description/urdf/naviton.urdf.xacro (robot description, xacro)
@@ -38,5 +38,5 @@
     <!-- LRF -->
     <xacro:lrf_v0 prefix="front" parent="base_link">
-  	    <origin xyz="0.155 0.0 0.195" rpy="${M_PI} 0 0"/>
+  	    <origin xyz="0.235 0.0 0.205" rpy="0 0 0"/>
     </xacro:lrf_v0>
     <xacro:lrf_gazebo_v0    topic_name="sensors/lrf/scan" prefix="front"
