Commit message: add naviton_v2 as new model

File: naviton/nvt_description/urdf/wheel/wheel.urdf.xacro (robot description, xacro)
@@ -22,5 +22,5 @@
                 </material>
 	        </visual>
-            <collision>
+          <collision>
 		        <origin xyz="0 -0.003 0" rpy="${-M_PI/2} 0 0"/>
 		        <geometry>
@@ -28,5 +28,5 @@
 		        </geometry>
 	        </collision>
-            <inertial>
+          <inertial>
 		        <origin xyz="0 -0.003 0" rpy="${-M_PI/2} 0 0"/>
 		        <xacro:cylinder_inertia mass="${wheel_mass}"
